File: vending-machine/electronic-design/vending-machine/vending-machine.kicad_pcb (KiCad board)
At the start: 2 copper layers, 40 parts, among them J1 Raspberry_Pi_2_3, J2 12V Input, J3 12V Output, J4 5V Input, J5 Conn_01x03_Male, J6 Conn_01x03_Male, J7 Conn_01x03_Male, M1 Stepper_Motor_unipolar_5pin, M2 Stepper_Motor_unipolar_5pin, M3 Stepper_Motor_unipolar_6pin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

Commit message: Schematic design
Parts:
- moved P1 31.8 mm to (125.8, 54.6)
Changed lines of the file:
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@@
   )
   (footprint "Connector_PinSocket_2.54mm:PinSocket_1x08_P2.54mm_Vertical" (layer "F.Cu")
-    (at 157.48 53.34)
+    (at 125.755 54.625)
     (descr "Through hole straight socket strip, 1x08, 2.54mm pitch, single row (from Kicad 4.0.7), script generated")
     (tags "Through hole socket strip THT 1x08 2.54mm single row")
