File: vending-machine/electronic-design/vending-machine-w-headers/vending-machine.kicad_pcb (KiCad board)
At the start: 2 copper layers, 40 parts, among them J1 Raspberry_Pi_4, J10 Motor, J2 12V Input, J3 12V Output, J4 5V Input, J5 Conn_01x03_Male, J6 Conn_01x03_Male, J7 Conn_01x03_Male, J8 Motor, J9 Motor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

Commit message: Vending machine PDB final design
Parts:
- added REF**: PinHeader_1x04_P2.54mm_Vertical, Connector_PinHeader_2.54mm:PinHeader_1x04_P2.54mm_Vertical, F.Cu at (37.6, 97.8)
- added REF**: PinHeader_1x04_P2.54mm_Vertical, Connector_PinHeader_2.54mm:PinHeader_1x04_P2.54mm_Vertical, F.Cu at (37.5, 34.4)
- added REF**: PinHeader_1x04_P2.54mm_Vertical, Connector_PinHeader_2.54mm:PinHeader_1x04_P2.54mm_Vertical, F.Cu at (37.5, 66.0)
- moved U2 2.42 mm to (85.2, 33.1)
- moved U1 2.16 mm to (69.0, 32.9)
- moved C15 1.74 mm to (66.3, 45.3)
Routing:
- net Net-(J8-Pad4): track 18.4 -> 29.1 mm
- net Net-(J9-Pad4): track 18.4 -> 29.0 mm
- net Net-(J10-Pad4): track 18.4 -> 29.0 mm
- net Net-(J8-Pad3): track 17.3 -> 24.5 mm
- net Net-(J10-Pad3): track 17.3 -> 24.4 mm
- net Net-(J9-Pad3): track 17.3 -> 24.4 mm
- net +12V: track 258.0 -> 263.1 mm
- net Net-(J8-Pad2): track 16.3 -> 19.8 mm
- net Net-(J9-Pad2): track 16.3 -> 19.7 mm
- net Net-(J10-Pad2): track 16.3 -> 19.7 mm
- net V Sensor: track 36.7 -> 39.3 mm
- net H Sensor: track 64.8 -> 63.6 mm
- net +3V3: track 55.8 -> 56.3 mm
