File: vending-machine/electronic-design/vending-machine-w-headers/vending-machine.kicad_sch (KiCad schematic)
At the start: 40 parts, among them J1 Raspberry_Pi_2_3, J2 12V Input, J3 12V Output, J4 5V Input, J5 Conn_01x03_Male, J6 Conn_01x03_Male, J7 Conn_01x03_Male, M1 Stepper_Motor_unipolar_5pin, M2 Stepper_Motor_unipolar_5pin, M3 Stepper_Motor_unipolar_6pin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

Commit message: Schematic design
Parts:
- removed M3, M4, M5: Stepper_Motor_unipolar_6pin, TerminalBlock:TerminalBlock_bornier-6_P5.08mm, symbol Motor:Stepper_Motor_unipolar_6pin
- added C15, C16, C17: 100n, Capacitor_THT:C_Disc_D6.0mm_W4.4mm_P5.00mm, symbol Device:C_Small
- added J10, J8, J9: Motor, TerminalBlock:TerminalBlock_bornier-4_P5.08mm, symbol Connector:Screw_Terminal_01x04
- J1: value Raspberry_Pi_2_3 -> Raspberry_Pi_4
- M1, M2: footprint TerminalBlock:TerminalBlock_bornier-6_P5.08mm -> TerminalBlock:TerminalBlock_bornier-5_P5.08mm
- P1: footprint Connector_PinSocket_2.54mm:PinSocket_1x08_P2.54mm_Vertical -> Connector_PinHeader_2.54mm:PinHeader_1x08_P2.54mm_Vertical
Connections:
- net +3V3: now also U1.1 (VCC), U2.1 (VCC); no longer U1. (VCC), U2. (VCC)
- net D CNTRL I1: now also J1.32 (PWM0/GPIO12); no longer J1.35 (GPIO19/MISO1)
- net D CNTRL I2: now also J1.36 (GPIO16); no longer J1.38 (GPIO20/MOSI1)
- net D CNTRL I3: now also J1.38 (GPIO20/MOSI1); no longer J1.40 (GPIO21/SCLK1)
- net D CNTRL I4: now also J1.40 (GPIO21/SCLK1); no longer J1.15 (GPIO22)
- net DIR CNTRL: now also J1.13 (GPIO27); no longer J1.3 (SDA/GPIO2)
- net EN CNTRL: now also J1.11 (GPIO17); no longer J1.5 (SCL/GPIO3)
- net GND: now also P1.4 (GND), U1.2 (GND), U2.2 (GND), C15.1, C16.1, C17.1; no longer P1.6 (GND), U1. (VCC), U2. (VCC)
- net H STEP CNTRL: now also J1.7 (GCLK0/GPIO4), C15.2; no longer J1.27 (ID_SD/GPIO0)
- net H Sensor: now also J1.5 (SCL/GPIO3), U2.3 (SIG); no longer J1.12 (GPIO18/PWM0), U2. (VCC)
- net Limit SW: now also J1.18 (GPIO24); no longer J1.36 (GPIO16)
- net PD CNTRL I1: now also J1.37 (GPIO26); no longer J1.16 (GPIO23)
- net PD CNTRL I2: now also J1.35 (GPIO19/MISO1); no longer J1.18 (GPIO24)
- net PD CNTRL I3: now also J1.33 (PWM1/GPIO13); no longer J1.22 (GPIO25)
- net PD CNTRL I4: now also J1.31 (GCLK2/GPIO6); no longer J1.37 (GPIO26)
- net V STEP CNTRL: now also J1.15 (GPIO22), C16.2, C17.2; no longer J1.28 (ID_SC/GPIO1)
- net V Sensor: now also J1.3 (SDA/GPIO2), U1.3 (SIG); no longer J1.11 (GPIO17), U1. (VCC)
- net RFID MOSI: now reaches J1.19 (MOSI0/GPIO10)
- net RFID MOSI: now also P1.7 (MOSI); no longer P1.3 (MOSI)
- net RFID MISO: now reaches J1.21 (MISO0/GPIO9)
- net RFID MISO: now also P1.6 (MISO); no longer P1.4 (MISO)
- net at P1.2 (IRQ): no longer J1.23 (SCLK0/GPIO11)
- net RFID SDA: now reaches J1.24 (~{CE0}/GPIO8), P1.1 (SDA)
- net RFID RST: now reaches J1.29 (GCLK1/GPIO5)
- net RFID RST: now also P1.3 (RST)
- net at U4.5 (2A): now also J9.2 (Pin_2)
- net at U4.6 (2B): now also J9.1 (Pin_1)
- net at U4.4 (1A): now also J9.3 (Pin_3)
- net at U4.3 (IB): now also J9.4 (Pin_4)
- net at U7.3 (IB): now also J10.4 (Pin_4)
- net at U7.4 (1A): now also J10.3 (Pin_3)
- net at U7.5 (2A): now also J10.2 (Pin_2)
- net at U7.6 (2B): now also J10.1 (Pin_1)
- net RFID SCK: now reaches P1.5 (SCK)
- net RFID SCK: now also J1.23 (SCLK0/GPIO11)
- net at U3.5 (2A): now also J8.2 (Pin_2)
- net at U3.6 (2B): now also J8.1 (Pin_1)
- net at U3.4 (1A): now also J8.3 (Pin_3)
- net at U3.3 (IB): now also J8.4 (Pin_4)
- no-connect marks 32 -> 27
Other:
- note added: "NFC Reader"
